Commit message: Major refactory of the repository : The name of the packgae was changed from iss_description to simulator_ros2 1)Launch files were modified to accomodate changing the target and the chaser model 2)Added the Aurora model as target spacerfat to be applied fo simulation 3) updated package.xml to include dependencies on simulator_msgs

File: description/ISS/urdf/model/model.xacro (robot description, xacro)
@@ -1,4 +1,4 @@
 <?xml version="1.0"?>
-<robot name="iss" xmlns:xacro="http://ros.org/wiki/xacro">
+<robot name="ISS" xmlns:xacro="http://ros.org/wiki/xacro">
   <xacro:property name="PI" value="3.1415926535897931" />
   <link name="fixed_link"/>
@@ -7,7 +7,6 @@
       <origin xyz="0 0 0" rpy="0 0 ${PI}" />
       <geometry>
-        <mesh filename="file://$(find iss_description)/description/meshes/ISS_2016.stl" scale="0.01 0.01 0.01"/>
+        <mesh filename="file://$(find simulator_ros2)/description/ISS/meshes/ISS_2016.stl" scale="0.01 0.01 0.01"/>
       </geometry>
-      <material name="yellow" />
     </visual>
     <inertial>
